Commit message: 修改接收器信息

File: usv_hardware/description/usv_core.xacro (robot description, xacro)
@@ -21,23 +21,4 @@
         <geometry>
           <box size="1 1 0.1"/>
-        </geometry>
-      </collision>
-    </link>
-    <!-- odom -->
-    <joint name="odom" type="fixed">
-      <parent link="odom"/>
-      <child link="base_link"/>
-      <origin xyz="0 0 0" rpy="0 0 0"/>
-    </joint>
-    <!-- Odom Link -->
-    <link name="odom">
-      <visual>
-        <geometry>
-          <box size="0.1 0.1 0.1"/>
-        </geometry>
-      </visual>
-      <collision>
-        <geometry>
-          <box size="0.1 0.1 0.1"/>
         </geometry>
       </collision>

Commit message: 仅软件测试

File: usv_hardware/description/usv_core.xacro (robot description, xacro)
@@ -24,4 +24,10 @@
       </collision>
     </link>
+    <joint name="magnetometer_joint" type="fixed">
+      <parent link="base_link"/>
+      <child link="magnetometer_link"/>
+      <origin xyz="0 0 0" rpy="0 0 -1.5708" /> <!-- RPY中的 -1.5708 约等于 -90度 -->
+    </joint>
+    <link name="magnetometer_link"></link>
     <joint name="laser" type="fixed">
       <parent link="base_footprint"/>
